Commit message: DexPilot and Mink baselines, run through their upstream libraries
Both baselines call the original authors' packages (dex_retargeting, mink); we
supply only the per-robot configuration, which lives in configs/baselines/ in
full view.  A baseline we reimplemented ourselves would not be worth comparing
against.

Neither method places the wrist, so both get the same treatment: DexPilot's
joint solution is positioned by a Kabsch fit of all 21 robot keypoints onto the
human's, and Mink is given a <freejoint> so it solves the base pose and the
joint angles together -- the strongest form of each, rather than handing them
the human wrist pose.

Two asset problems surfaced and are fixed:

- the vendored URDF still said ../meshes/, correct upstream where the URDF sits
  in urdf/, wrong here where it sits beside meshes/.  Only mesh loaders noticed,
  so pytorch_kinematics and our own pipeline had masked it.
- MuJoCo merges fixed-joint links into their parent, so the five *_tip_link
  frames our keypoint correspondence needs do not exist as bodies in the MJCF.
  They are recovered as sites, with the offsets read from the URDF's fixed
  joints (all five are pure translations; a non-zero rpy raises rather than
  silently dropping the rotation).

First real comparison, ContactPose full28_use/mug, before any tuning:
  ours     E_prec  5.59 mm   D_pen_max 3.21 mm   18.9 s
  mink     E_prec  5.80 mm   D_pen_max 4.97 mm    0.08 s
  dexpilot E_prec 12.84 mm   D_pen_max 5.47 mm    0.05 s

File: assets/wuji_right/right.urdf (robot description, URDF)
Before this commit: robot wujihand-right, 26 links, 25 joints
Links:
- link right_finger1_link1: geometry collision mesh filename=meshes/right_finger1_link1.STL; visual mesh filename=meshes/right_finger1_link1.STL
- link right_finger1_link2: geometry collision mesh filename=meshes/right_finger1_link2.STL; visual mesh filename=meshes/right_finger1_link2.STL
- link right_finger1_link3: geometry collision mesh filename=meshes/right_finger1_link3.STL; visual mesh filename=meshes/right_finger1_link3.STL
- link right_finger1_link4: geometry collision mesh filename=meshes/right_finger1_link4.STL; visual mesh filename=meshes/right_finger1_link4.STL
- link right_finger1_tip_link: geometry collision mesh filename=meshes/right_finger1_tip_link.STL; visual mesh filename=meshes/right_finger1_tip_link.STL
- link right_finger2_link1: geometry collision mesh filename=meshes/right_finger2_link1.STL; visual mesh filename=meshes/right_finger2_link1.STL
- link right_finger2_link2: geometry collision mesh filename=meshes/right_finger2_link2.STL; visual mesh filename=meshes/right_finger2_link2.STL
- link right_finger2_link3: geometry collision mesh filename=meshes/right_finger2_link3.STL; visual mesh filename=meshes/right_finger2_link3.STL
- link right_finger2_link4: geometry collision mesh filename=meshes/right_finger2_link4.STL; visual mesh filename=meshes/right_finger2_link4.STL
- link right_finger2_tip_link: geometry collision mesh filename=meshes/right_finger2_tip_link.STL; visual mesh filename=meshes/right_finger2_tip_link.STL
- link right_finger3_link1: geometry collision mesh filename=meshes/right_finger3_link1.STL; visual mesh filename=meshes/right_finger3_link1.STL
- link right_finger3_link2: geometry collision mesh filename=meshes/right_finger3_link2.STL; visual mesh filename=meshes/right_finger3_link2.STL
- link right_finger3_link3: geometry collision mesh filename=meshes/right_finger3_link3.STL; visual mesh filename=meshes/right_finger3_link3.STL
- link right_finger3_link4: geometry collision mesh filename=meshes/right_finger3_link4.STL; visual mesh filename=meshes/right_finger3_link4.STL
- link right_finger3_tip_link: geometry collision mesh filename=meshes/right_finger3_tip_link.STL; visual mesh filename=meshes/right_finger3_tip_link.STL
- link right_finger4_link1: geometry collision mesh filename=meshes/right_finger4_link1.STL; visual mesh filename=meshes/right_finger4_link1.STL
- link right_finger4_link2: geometry collision mesh filename=meshes/right_finger4_link2.STL; visual mesh filename=meshes/right_finger4_link2.STL
- link right_finger4_link3: geometry collision mesh filename=meshes/right_finger4_link3.STL; visual mesh filename=meshes/right_finger4_link3.STL
- link right_finger4_link4: geometry collision mesh filename=meshes/right_finger4_link4.STL; visual mesh filename=meshes/right_finger4_link4.STL
- link right_finger4_tip_link: geometry collision mesh filename=meshes/right_finger4_tip_link.STL; visual mesh filename=meshes/right_finger4_tip_link.STL
- link right_finger5_link1: geometry collision mesh filename=meshes/right_finger5_link1.STL; visual mesh filename=meshes/right_finger5_link1.STL
- link right_finger5_link2: geometry collision mesh filename=meshes/right_finger5_link2.STL; visual mesh filename=meshes/right_finger5_link2.STL
- link right_finger5_link3: geometry collision mesh filename=meshes/right_finger5_link3.STL; visual mesh filename=meshes/right_finger5_link3.STL
- link right_finger5_link4: geometry collision mesh filename=meshes/right_finger5_link4.STL; visual mesh filename=meshes/right_finger5_link4.STL
- link right_finger5_tip_link: geometry collision mesh filename=meshes/right_finger5_tip_link.STL; visual mesh filename=meshes/right_finger5_tip_link.STL
- link right_palm_link: geometry collision mesh filename=meshes/right_palm_link.STL; visual mesh filename=meshes/right_palm_link.STL
